Commit message: Novel dataset3 with new initial estimate.

File: nrp_calibration/urdf/initial_estimate.urdf.xacro (robot description, xacro)
@@ -1,42 +1,44 @@
-<?xml version="1.0"?>
-<robot name="arm_with_effector" xmlns:xacro="http://ros.org/wiki/xacro">
-    <link name="world"/>
-    <link name="link1"/>
-    <link name="link2"/>
-    <link name="camera1_link"/>
-    <link name="camera2_link"/>
-    <link name="marker_link" />
-    <link name="camera1_color_optical_frame" />
-    <link name="camera2_color_optical_frame" />
-    <joint name="world_link1_joint" type="fixed">
-        <origin xyz="0.1 -0.2 0.3" rpy="0 0 1.57"/>
-        <parent link="world"/>
-        <child link="link1"/>
-    </joint>
-    <joint name="world_link2_joint" type="fixed">
-        <origin xyz="-0.1 -0.2 0.3" rpy="0 0 1.57"/>
-        <parent link="world"/>
-        <child link="link2"/>
-    </joint>
-    <joint name="link1_camera1_joint" type="fixed">
-        <parent link="link1"/>
-        <child link="camera1_link"/>
-    </joint>
-    <joint name="link2_camera1_joint" type="fixed">
-        <parent link="link2"/>
-        <child link="camera2_link"/>
-    </joint>
-    <joint name="link1_camera1_optical_joint" type="fixed">
-        <parent link="camera1_link"/>
-        <child link="camera1_color_optical_frame"/>
-    </joint>
-    <joint name="link2_camera2_optical_joint" type="fixed">
-        <parent link="camera2_link"/>
-        <child link="camera2_color_optical_frame"/>
-    </joint>
-     <joint name="world_marker_joint" type="fixed">
-        <origin xyz="0.0 0.2 0.3" rpy="1.57 0 0"/>
-        <parent link="world"/>
-        <child link="marker_link"/>
-    </joint>
+<?xml version="1.0" ?>
+<robot name="arm_with_effector" version="1.0">
+  <link name="world"/>
+  <link name="link1"/>
+  <link name="link2"/>
+  <link name="camera1_link"/>
+  <link name="camera2_link"/>
+  <link name="marker_link"/>
+  <link name="camera1_color_optical_frame"/>
+  <link name="camera2_color_optical_frame"/>
+  <joint name="world_link1_joint" type="fixed">
+    <origin xyz="0.1 -0.2 0.3" rpy="0.0 0.0 1.57"/>
+    <parent link="world"/>
+    <child link="link1"/>
+  </joint>
+  <joint name="world_link2_joint" type="fixed">
+    <origin xyz="-0.1 -0.2 0.3" rpy="0.0 0.0 1.57"/>
+    <parent link="world"/>
+    <child link="link2"/>
+  </joint>
+  <joint name="link1_camera1_joint" type="fixed">
+    <origin xyz="0.0 0.0 0.0" rpy="0.0 -0.0 0.0"/>
+    <parent link="link1"/>
+    <child link="camera1_link"/>
+  </joint>
+  <joint name="link2_camera1_joint" type="fixed">
+    <origin xyz="-1.4192314147949219 -0.21051329374313354 0.0" rpy="0.0 -0.0 0.0"/>
+    <parent link="link2"/>
+    <child link="camera2_link"/>
+  </joint>
+  <joint name="link1_camera1_optical_joint" type="fixed">
+    <parent link="camera1_link"/>
+    <child link="camera1_color_optical_frame"/>
+  </joint>
+  <joint name="link2_camera2_optical_joint" type="fixed">
+    <parent link="camera2_link"/>
+    <child link="camera2_color_optical_frame"/>
+  </joint>
+  <joint name="world_marker_joint" type="fixed">
+    <origin xyz="0.0 0.2 0.3" rpy="1.57 0.0 0.0"/>
+    <parent link="world"/>
+    <child link="marker_link"/>
+  </joint>
 </robot>

Commit message: Updating the dataset3 with a better initial estimate.

File: nrp_calibration/urdf/initial_estimate.urdf.xacro (robot description, xacro)
@@ -25,5 +25,5 @@
   </joint>
   <joint name="link2_camera1_joint" type="fixed">
-    <origin xyz="-1.4192314147949219 -0.21051329374313354 0.0" rpy="0.0 -0.0 0.0"/>
+    <origin xyz="-0.4271034002304077 -0.18467563390731812 0.0" rpy="0.0 -0.0 0.0"/>
     <parent link="link2"/>
     <child link="camera2_link"/>

File: nrp_calibration/urdf/optimized/optimized_2023_04_19-01_07_06_AM.urdf.xacro (robot description, xacro)
@@ -20,10 +20,10 @@
   </joint>
   <joint name="link1_camera1_joint" type="fixed">
-    <origin xyz="-0.08989991335059389 0.011578726685219426 -0.08948315822909549" rpy="-0.0747317906367676 -0.10457966156657274 0.2414603238921311"/>
+    <origin xyz="-0.10427068671764803 0.02988901056264166 -0.08816714524916303" rpy="0.044495448923149265 -0.12881068198040357 -0.05816276430069011"/>
     <parent link="link1"/>
     <child link="camera1_link"/>
   </joint>
   <joint name="link2_camera1_joint" type="fixed">
-    <origin xyz="-0.41578142644908084 -0.18801862343883347 -0.003166817419593214" rpy="-0.0179530877957564 0.02207522257944473 0.1039402446237512"/>
+    <origin xyz="-0.42264703731726816 -0.18293624072242406 0.040877989302344486" rpy="-0.008361261900862942 0.009752340777105153 0.013200861312459216"/>
     <parent link="link2"/>
     <child link="camera2_link"/>

File: nrp_calibration/urdf/optimized/optimized_2023_04_19-12_51_57_AM.urdf.xacro (robot description, xacro)
@@ -20,10 +20,10 @@
   </joint>
   <joint name="link1_camera1_joint" type="fixed">
-    <origin xyz="-0.08989991335059389 0.011578726685219426 -0.08948315822909549" rpy="-0.0747317906367676 -0.10457966156657274 0.2414603238921311"/>
+    <origin xyz="-4.440892098498797e-16 -1.3953037152288693e-16 -4.4375157641055787e-16" rpy="3.795934752968473e-16 -4.406743123681939e-16 4.3604063938477617e-16"/>
     <parent link="link1"/>
     <child link="camera1_link"/>
   </joint>
   <joint name="link2_camera1_joint" type="fixed">
-    <origin xyz="-0.41578142644908084 -0.18801862343883347 -0.003166817419593214" rpy="-0.0179530877957564 0.02207522257944473 0.1039402446237512"/>
+    <origin xyz="-1.2322489875842622 -0.18734855247360432 0.08002238878242166" rpy="0.6056921156482382 0.41385910989909025 0.898514937869043"/>
     <parent link="link2"/>
     <child link="camera2_link"/>

File: nrp_calibration/urdf/optimized/optimized_2023_04_19-12_59_34_AM.urdf.xacro (robot description, xacro)
@@ -20,10 +20,10 @@
   </joint>
   <joint name="link1_camera1_joint" type="fixed">
-    <origin xyz="-0.08989991335059389 0.011578726685219426 -0.08948315822909549" rpy="-0.0747317906367676 -0.10457966156657274 0.2414603238921311"/>
+    <origin xyz="-0.1101270771735845 -0.20216576707684192 0.03694997511211755" rpy="-0.44567887580764565 0.007194976373170318 0.36878255853139985"/>
     <parent link="link1"/>
     <child link="camera1_link"/>
   </joint>
   <joint name="link2_camera1_joint" type="fixed">
-    <origin xyz="-0.41578142644908084 -0.18801862343883347 -0.003166817419593214" rpy="-0.0179530877957564 0.02207522257944473 0.1039402446237512"/>
+    <origin xyz="-0.3820019415284816 -0.23839103077501073 -0.02565416002242052" rpy="0.0258083559295182 0.021128058264670225 0.37006693699153803"/>
     <parent link="link2"/>
     <child link="camera2_link"/>

Commit message: Found the issue. Added dataset4 with pattern not fixed.

File: nrp_calibration/urdf/initial_estimate.urdf.xacro (robot description, xacro)
@@ -20,10 +20,10 @@
   </joint>
   <joint name="link1_camera1_joint" type="fixed">
-    <origin xyz="0.0 0.0 0.0" rpy="0.0 -0.0 0.0"/>
+    <origin xyz="0.5540721416473389 0.19767163693904877 0.0" rpy="0.0 -0.0 0.0"/>
     <parent link="link1"/>
     <child link="camera1_link"/>
   </joint>
   <joint name="link2_camera1_joint" type="fixed">
-    <origin xyz="-0.4271034002304077 -0.18467563390731812 0.0" rpy="0.0 -0.0 0.0"/>
+    <origin xyz="0.0 0.0 0.0" rpy="0.0 -0.0 0.0"/>
     <parent link="link2"/>
     <child link="camera2_link"/>

File: nrp_calibration/urdf/optimized/optimized_2023_04_19-01_16_11_AM.urdf.xacro (robot description, xacro)
@@ -20,10 +20,10 @@
   </joint>
   <joint name="link1_camera1_joint" type="fixed">
-    <origin xyz="-0.10185413390876669 -0.242730281795217 0.04317593204980823" rpy="-0.5223655953853976 0.03192681993488331 0.3877203722497517"/>
+    <origin xyz="-0.09896468751134616 0.12148757520269639 0.018863015938360133" rpy="0.3022600167319036 -0.10302127368538945 -0.2137819347579142"/>
     <parent link="link1"/>
     <child link="camera1_link"/>
   </joint>
   <joint name="link2_camera1_joint" type="fixed">
-    <origin xyz="-0.3845053464933208 -0.24025312362980633 -0.02795309174630628" rpy="0.03874160622700417 0.021067395521222068 0.3958297165414839"/>
+    <origin xyz="-0.38776389162952374 -0.17105195567813877 -0.004064008398568736" rpy="-0.032743622766574304 0.045379510708752714 -0.23668380348163312"/>
     <parent link="link2"/>
     <child link="camera2_link"/>

File: nrp_calibration/urdf/optimized/optimized_2023_04_20-08_06_28_PM.urdf.xacro (robot description, xacro)
@@ -20,10 +20,10 @@
   </joint>
   <joint name="link1_camera1_joint" type="fixed">
-    <origin xyz="-0.10185413390876669 -0.242730281795217 0.04317593204980823" rpy="-0.5223655953853976 0.03192681993488331 0.3877203722497517"/>
+    <origin xyz="-0.09896470062287113 0.12148747223208176 0.01886310038364904" rpy="0.3022598104302074 -0.10302134128621819 -0.21378163173771264"/>
     <parent link="link1"/>
     <child link="camera1_link"/>
   </joint>
   <joint name="link2_camera1_joint" type="fixed">
-    <origin xyz="-0.3845053464933208 -0.24025312362980633 -0.02795309174630628" rpy="0.03874160622700417 0.021067395521222068 0.3958297165414839"/>
+    <origin xyz="-0.38776384816198123 -0.17105191753456825 -0.004064037285265582" rpy="-0.03274339406236669 0.04537945882084853 -0.2366834073834174"/>
     <parent link="link2"/>
     <child link="camera2_link"/>

File: nrp_calibration/urdf/optimized/optimized_2023_04_20-08_08_19_PM.urdf.xacro (robot description, xacro)
@@ -20,10 +20,10 @@
   </joint>
   <joint name="link1_camera1_joint" type="fixed">
-    <origin xyz="-0.10185413390876669 -0.242730281795217 0.04317593204980823" rpy="-0.5223655953853976 0.03192681993488331 0.3877203722497517"/>
+    <origin xyz="-0.10185515865401772 -0.2427293353963351 0.043178434440970484" rpy="-0.522367149856401 0.03192728600252762 0.3877217856257287"/>
     <parent link="link1"/>
     <child link="camera1_link"/>
   </joint>
   <joint name="link2_camera1_joint" type="fixed">
-    <origin xyz="-0.3845053464933208 -0.24025312362980633 -0.02795309174630628" rpy="0.03874160622700417 0.021067395521222068 0.3958297165414839"/>
+    <origin xyz="-0.3845050166413971 -0.24025320223588223 -0.02795579686821271" rpy="0.03874300004986609 0.02106713896501689 0.3958320171184378"/>
     <parent link="link2"/>
     <child link="camera2_link"/>
